Commit message: working version both in simulation and on the real robot

File: config/panda_arm.xacro (robot description, xacro)
@@ -9,4 +9,7 @@
     <group name="panda_arm">
       <chain base_link="panda_link0" tip_link="panda_link8" />
+    </group>
+    <group name="panda_end_effector">
+        <link name="panda_link8"/>
     </group>
     <!--GROUP STATES: Purpose: Define a named state for a particular group, in terms of joint values. This is useful to define states like 'folded arms'-->
@@ -21,6 +24,7 @@
     </group_state>
     <!--END EFFECTOR: Purpose: Represent information about an end effector.-->
+    <end_effector name="panda_arm_ee" parent_link="panda_link8" group="panda_end_effector" parent_group="panda_arm" />
     <!--VIRTUAL JOINT: Purpose: this element defines a virtual joint between a robot link and an external frame of reference (considered fixed with respect to the robot)-->
-    <virtual_joint name="virtual_joint" type="floating" parent_frame="world" child_link="panda_link0" />
+    <!-- <virtual_joint name="virtual_joint" type="floating" parent_frame="world" child_link="panda_link0" /> -->
     <!--DISABLE COLLISIONS: By default it is assumed that any link of the robot could potentially come into collision with any other link in the robot. This tag disables collision checking between a specified pair of links. -->
     <disable_collisions link1="panda_link0" link2="panda_link1" reason="Adjacent" />
