Commit message: add gripper control

File: config/hand.xacro (robot description, xacro)
@@ -12,5 +12,5 @@
       <link name="panda_rightfinger" />
       <joint name="panda_finger_joint1" />
-      <passive_joint name="panda_finger_joint2" />
+      <joint name="panda_finger_joint2" />
     </group>
     <!--GROUP STATES: Purpose: Define a named state for a particular group, in terms of joint values. This is useful to define states like 'folded arms'-->
